File: DesignDocuments/osps/processor.sch (KiCad schematic (older format))
At the start: 3 parts

Commit message: make sure library links made
Parts:
- removed IC?: STM32F302R8T6, QFP50P1200X1200X160-64N, symbol STM32F302R8T6
- removed R? (x2): CRCW060310K0FKEA, RESC1608X55, symbol CRCW060310K0FKEA
- added IC?: STM32F302R8T6, QFP50P1200X1200X160-64N, symbol STM32F302R8T6
- added R? (x2): CRCW060310K0FKEA, RESC1608X55, symbol CRCW060310K0FKEA
Connections:
- net +3V3: now also R?.1
- net GND: now also IC?.12 (VSSA), IC?.18 (VSS_4), IC?.31 (VSS_2), IC?.47 (VSS_3), IC?.63 (VSS_1), R?.2
- new net: IC?.60 (BOOT0), R?.1
- new net: IC?.7 (!RST), R?.2
Changed lines of the file:
@@
 LIBS:CRCW060310K0FKEA
 LIBS:STM32F302R8T6
+LIBS:osps-cache
 EELAYER 25 0
 EELAYER END
 $Descr A4 11693 8268
 encoding utf-8
-Sheet 1 1
+Sheet 2 2
 Title ""
 Date ""
@@
 $Comp
 L STM32F302R8T6 IC?
-U 1 1 5785F90F
+U 1 1 5785F80A
 P 4850 3400
 F 0 "IC?" H 4450 5900 50  0000 L CNN
@@
 $Comp
 L CRCW060310K0FKEA R?
-U 1 1 5785F968
+U 1 1 5785F873
 P 2500 1400
 F 0 "R?" H 2350 1479 50  0000 L CNN
@@
 $Comp
 L CRCW060310K0FKEA R?
-U 1 1 5785F9B1
+U 1 1 5785F938
 P 2500 2300
 F 0 "R?" H 2350 2379 50  0000 L CNN

Commit message: added decopling to muc
Parts:
- removed R?: CRCW060310K0FKEA, RESC1608X55, symbol CRCW060310K0FKEA
- added C? (x5): 100nF, CAPC1608X90, symbol C0603C221J5GACTU
- added R?: 10K, RESC1608X55, symbol CRCW060310K0FKEA
- R?: value CRCW060310K0FKEA -> 10K; Package (none) -> 0603
Connections:
- wire segments 12 -> 29
Changed lines of the file:
@@
 LIBS:CRCW060310K0FKEA
 LIBS:STM32F302R8T6
-LIBS:osps-cache
+LIBS:C0603C221J5GACTU
 EELAYER 25 0
 EELAYER END
@@
 	1    0    0    -1
 $EndComp
-Wire Wire Line
-	5500 5800 5500 6350
-Wire Wire Line
-	5500 5800 5450 5800
-Wire Wire Line
-	5450 6200 5500 6200
-Connection ~ 5500 6200
-Wire Wire Line
-	5450 6100 5500 6100
-Connection ~ 5500 6100
-Wire Wire Line
-	5450 6000 5500 6000
-Connection ~ 5500 6000
-Wire Wire Line
-	5450 5900 5500 5900
-Connection ~ 5500 5900
 $Comp
 L GND #PWR?
@@
 	1    0    0    -1
 $EndComp
-Wire Wire Line
-	4250 1900 2500 1900
-Wire Wire Line
-	2500 1900 2500 2000
-Wire Wire Line
-	2500 2700 2500 2600
-Wire Wire Line
-	4250 1800 2500 1800
-Wire Wire Line
-	2500 1800 2500 1700
 $Comp
 L +3.3V #PWR?
@@
 	1    0    0    -1
 $EndComp
-Wire Wire Line
-	2500 1100 2500 1050
 $Comp
 L STM32F302R8T6 IC?
@@
 $Comp
 L CRCW060310K0FKEA R?
-U 1 1 5785F873
+U 1 1 5785F938
+P 2500 2300
+F 0 "R?" V 2350 2400 50  0000 L CNN
+F 1 "10K" V 2450 2400 50  0000 L CNN
+F 2 "RESC1608X55" H 2500 2300 50  0001 L CNN
+F 3 "" H 2500 2300 60  0000 C CNN
+F 4 "0603" V 2550 2500 60  0000 C CNN "Package"
+	1    2500 2300
+	0    1    1    0
+$EndComp
+$Comp
+L CRCW060310K0FKEA R?
+U 1 1 578689C1
 P 2500 1400
-F 0 "R?" H 2350 1479 50  0000 L CNN
-F 1 "CRCW060310K0FKEA" H 2350 1260 50  0000 L CNN
+F 0 "R?" V 2350 1500 50  0000 L CNN
+F 1 "10K" V 2450 1500 50  0000 L CNN
 F 2 "RESC1608X55" H 2500 1400 50  0001 L CNN
 F 3 "" H 2500 1400 60  0000 C CNN
+F 4 "0603" V 2550 1600 60  0000 C CNN "Package"
 	1    2500 1400
 	0    1    1    0
 $EndComp
-$Comp
-L CRCW060310K0FKEA R?
-U 1 1 5785F938
-P 2500 2300
-F 0 "R?" H 2350 2379 50  0000 L CNN
-F 1 "CRCW060310K0FKEA" H 2350 2160 50  0000 L CNN
-F 2 "RESC1608X55" H 2500 2300 50  0001 L CNN
-F 3 "" H 2500 2300 60  0000 C CNN
-	1    2500 2300
-	0    1    1    0
-$EndComp
+Wire Wire Line
+	5500 5800 5500 6350
+Wire Wire Line
+	5500 5800 5450 5800
+Wire Wire Line
+	5450 6200 5500 6200
+Connection ~ 5500 6200
+Wire Wire Line
+	5450 6100 5500 6100
+Connection ~ 5500 6100
+Wire Wire Line
+	5450 6000 5500 6000
+Connection ~ 5500 6000
+Wire Wire Line
+	5450 5900 5500 5900
+Connection ~ 5500 5900
+Wire Wire Line
+	4250 1900 2500 1900
+Wire Wire Line
+	2500 1900 2500 2000
+Wire Wire Line
+	2500 2700 2500 2600
+Wire Wire Line
+	4250 1800 2500 1800
+Wire Wire Line
+	2500 1800 2500 1700
+Wire Wire Line
+	2500 1100 2500 1050
+Wire Wire Line
+	5500 1500 5450 1500
+Connection ~ 5500 1400
+Connection ~ 5500 1300
+Connection ~ 5500 1200
+Wire Wire Line
+	5450 1100 8200 1100
+Connection ~ 5500 1500
+Wire Wire Line
+	5450 1400 5500 1400
+Wire Wire Line
+	5450 1300 5500 1300
+Wire Wire Line
+	5450 1200 5500 1200
+Wire Wire Line
+	5500 1100 5500 1500
+Wire Wire Line
+	6200 1100 6200 1150
+Connection ~ 5500 1100
+Wire Wire Line
+	6700 1100 6700 1150
+Connection ~ 6200 1100
+Wire Wire Line
+	7200 1100 7200 1150
+Connection ~ 6700 1100
+Wire Wire Line
+	7700 1100 7700 1150
+Connection ~ 7200 1100
+Wire Wire Line
+	8200 1100 8200 1150
+Connection ~ 7700 1100
+$Comp
+L C0603C221J5GACTU C?
+U 1 1 5786B50A
+P 6200 1350
+F 0 "C?" V 6100 1450 50  0000 L CNN
+F 1 "100nF" V 6200 1450 50  0000 L CNN
+F 2 "CAPC1608X90" H 6200 1350 50  0001 L CNN
+F 3 "" H 6200 1350 60  0000 C CNN
+F 4 "0603" V 6300 1550 60  0000 C CNN "Package"
+	1    6200 1350
+	0    1    1    0
+$EndComp
+$Comp
+L C0603C221J5GACTU C?
+U 1 1 5786B7B9
+P 6700 1350
+F 0 "C?" V 6600 1450 50  0000 L CNN
+F 1 "100nF" V 6700 1450 50  0000 L CNN
+F 2 "CAPC1608X90" H 6700 1350 50  0001 L CNN
+F 3 "" H 6700 1350 60  0000 C CNN
+F 4 "0603" V 6800 1550 60  0000 C CNN "Package"
+	1    6700 1350
+	0    1    1    0
+$EndComp
+$Comp
+L C0603C221J5GACTU C?
+U 1 1 5786B7F3
+P 7200 1350
+F 0 "C?" V 7100 1450 50  0000 L CNN
+F 1 "100nF" V 7200 1450 50  0000 L CNN
+F 2 "CAPC1608X90" H 7200 1350 50  0001 L CNN
+F 3 "" H 7200 1350 60  0000 C CNN
+F 4 "0603" V 7300 1550 60  0000 C CNN "Package"
+	1    7200 1350
+	0    1    1    0
+$EndComp
+$Comp
+L C0603C221J5GACTU C?
+U 1 1 5786B831
+P 7700 1350
+F 0 "C?" V 7600 1450 50  0000 L CNN
+F 1 "100nF" V 7700 1450 50  0000 L CNN
+F 2 "CAPC1608X90" H 7700 1350 50  0001 L CNN
+F 3 "" H 7700 1350 60  0000 C CNN
+F 4 "0603" V 7800 1550 60  0000 C CNN "Package"
+	1    7700 1350
+	0    1    1    0
+$EndComp
+$Comp
+L C0603C221J5GACTU C?
+U 1 1 5786B86D
+P 8200 1350
+F 0 "C?" V 8100 1450 50  0000 L CNN
+F 1 "100nF" V 8200 1450 50  0000 L CNN
+F 2 "CAPC1608X90" H 8200 1350 50  0001 L CNN
+F 3 "" H 8200 1350 60  0000 C CNN
+F 4 "0603" V 8300 1550 60  0000 C CNN "Package"
+	1    8200 1350
+	0    1    1    0
+$EndComp
+Wire Wire Line
+	8200 1550 8200 1600
+Wire Wire Line
+	8200 1600 6200 1600
+Wire Wire Line
+	6200 1600 6200 1550
+Wire Wire Line
+	6700 1550 6700 1600
+Connection ~ 6700 1600
+Wire Wire Line
+	7200 1550 7200 1600
+Connection ~ 7200 1600
+Wire Wire Line
+	7700 1550 7700 1600
+Connection ~ 7700 1600
 $EndSCHEMATC

Commit message: added ferrite, boot conf and caps
Parts:
- added F??: WURTH_ELEKTRONIK__742792651__FERRITE,_BEAD,_0603,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, symbol WURTH_ELEKTRONIK__742792651__FERRITE,_BEAD,_0603,_0.2OHM,_1A
- added R? (x2): 10K, RESC1608X55, symbol CRCW060310K0FKEA
- R? (x2): value 10K -> DNF
Connections:
- net labels added: BOOT0, NRST
- wire segments 29 -> 33
Other:
- note added: "BOOT0 = 0 - Flash\nBOOT0 = 1 - Bootloader"
- note added: "To reset processor short \nDNF pull down on NRST"
- moved on the sheet: R?

Commit message: added 24MHz osc
Parts:
- added C? (x2): 18pF, CAPC1608X90, symbol C0603C221J5GACTU
- added U?: ABLS-24.000MHZ-B4-T, XTAL1140X470X330, symbol ABLS2-8.000MHZ-D4Y-T
Connections:
- wire segments 33 -> 41
Changed lines of the file:
@@
 LIBS:C0603C221J5GACTU
 LIBS:wurth_742792651
+LIBS:ABLS2-8.000MHZ-D4Y-T
 LIBS:osps-cache
 EELAYER 25 0
@@
 Connection ~ 5500 1500
 Wire Wire Line
-	5450 1400 5500 1400
+	5500 1400 5450 1400
 Wire Wire Line
 	5450 1300 5500 1300
@@
 	7650 2050 7650 2150
 Wire Wire Line
-	7650 2100 5650 2100
+	5650 2100 7650 2100
 Wire Wire Line
 	5650 2100 5650 2050
@@
 $EndComp
 Wire Wire Line
-	7650 1600 5450 1600
+	5450 1600 7650 1600
 Connection ~ 5500 1600
 Wire Wire Line
@@
 Wire Wire Line
 	4250 1900 2150 1900
+$Comp
+L ABLS2-8.000MHZ-D4Y-T U?
+U 1 1 57870966
+P 6250 4500
+F 0 "U?" H 6500 4600 50  0000 L CNN
+F 1 "ABLS-24.000MHZ-B4-T" H 5650 4700 50  0000 L CNN
+F 2 "XTAL1140X470X330" H 6250 4500 50  0001 L CNN
+F 3 "" H 6250 4500 60  0000 C CNN
+	1    6250 4500
+	-1   0    0    1
+$EndComp
+$Comp
+L C0603C221J5GACTU C?
+U 1 1 5787143E
+P 6950 5050
+F 0 "C?" V 6850 5150 50  0000 L CNN
+F 1 "18pF" V 6950 5150 50  0000 L CNN
+F 2 "CAPC1608X90" H 6950 5050 50  0001 L CNN
+F 3 "" H 6950 5050 60  0000 C CNN
+F 4 "0603" V 7050 5250 60  0000 C CNN "Package"
+	1    6950 5050
+	0    1    1    0
+$EndComp
+$Comp
+L C0603C221J5GACTU C?
+U 1 1 578711C8
+P 5650 5050
+F 0 "C?" V 5550 5150 50  0000 L CNN
+F 1 "18pF" V 5650 5150 50  0000 L CNN
+F 2 "CAPC1608X90" H 5650 5050 50  0001 L CNN
+F 3 "" H 5650 5050 60  0000 C CNN
+F 4 "0603" V 5750 5250 60  0000 C CNN "Package"
+	1    5650 5050
+	0    1    1    0
+$EndComp
+Wire Wire Line
+	5450 4500 5950 4500
+Wire Wire Line
+	5650 5400 6950 5400
+Wire Wire Line
+	6950 4400 6950 4850
+Wire Wire Line
+	5450 4400 6950 4400
+Wire Wire Line
+	6950 4500 6550 4500
+Connection ~ 6950 4500
+Wire Wire Line
+	6950 5250 6950 5500
+$Comp
+L GND #PWR?
+U 1 1 578728D5
+P 6950 5500
+F 0 "#PWR?" H 6950 5250 50  0001 C CNN
+F 1 "GND" H 6950 5350 50  0000 C CNN
+F 2 "" H 6950 5500 50  0000 C CNN
+F 3 "" H 6950 5500 50  0000 C CNN
+	1    6950 5500
+	1    0    0    -1
+$EndComp
+Connection ~ 6950 5400
+Wire Wire Line
+	5650 4850 5650 4500
+Connection ~ 5650 4500
+Wire Wire Line
+	5650 5400 5650 5250
 $EndSCHEMATC

Commit message: added debug header
Parts:
- added U?: Header,7x1,2.54mm, symbol Header,7x1,2.54mm
Connections:
- net labels added: SYS_JTCK-SWCLK, SYS_JTDI, SYS_JTDO-TRACESWO, SYS_JTMS-SWDIO, SYS_NJTRST
- wire segments 41 -> 77
Changed lines of the file:
@@
 LIBS:wurth_742792651
 LIBS:ABLS2-8.000MHZ-D4Y-T
+LIBS:header-7x1-254
+LIBS:header-3x1-254
 LIBS:osps-cache
 EELAYER 25 0
@@
 	0    1    1    0
 $EndComp
-Wire Wire Line
-	5500 5800 5500 6350
-Wire Wire Line
-	5500 5800 5450 5800
-Wire Wire Line
-	5450 6200 5500 6200
-Connection ~ 5500 6200
-Wire Wire Line
-	5450 6100 5500 6100
-Connection ~ 5500 6100
-Wire Wire Line
-	5450 6000 5500 6000
-Connection ~ 5500 6000
-Wire Wire Line
-	5450 5900 5500 5900
-Connection ~ 5500 5900
-Wire Wire Line
-	2650 1650 2650 2000
-Wire Wire Line
-	2650 2700 2650 2600
-Wire Wire Line
-	2150 1650 2150 2000
-Wire Wire Line
-	2150 1050 2150 1000
-Wire Wire Line
-	5500 1500 5450 1500
-Connection ~ 5500 1400
-Connection ~ 5500 1300
-Connection ~ 5500 1500
-Wire Wire Line
-	5500 1400 5450 1400
-Wire Wire Line
-	5450 1300 5500 1300
-Wire Wire Line
-	5450 1200 5500 1200
-Wire Wire Line
-	5650 1600 5650 1650
-Wire Wire Line
-	6150 1600 6150 1650
-Connection ~ 5650 1600
-Wire Wire Line
-	6650 1600 6650 1650
-Connection ~ 6150 1600
-Wire Wire Line
-	7150 1600 7150 1650
-Connection ~ 6650 1600
-Wire Wire Line
-	7650 1050 7650 1650
-Connection ~ 7150 1600
 $Comp
 L C0603C221J5GACTU C?
@@
 	0    1    1    0
 $EndComp
-Wire Wire Line
-	7650 2050 7650 2150
-Wire Wire Line
-	5650 2100 7650 2100
-Wire Wire Line
-	5650 2100 5650 2050
-Wire Wire Line
-	6150 2050 6150 2100
-Connection ~ 6150 2100
-Wire Wire Line
-	6650 2050 6650 2100
-Connection ~ 6650 2100
-Wire Wire Line
-	7150 2050 7150 2100
-Connection ~ 7150 2100
 $Comp
 L WURTH_ELEKTRONIK__742792651__FERRITE,_BEAD,_0603,_0.2OHM,_1A F??
@@
 	1    0    0    -1
 $EndComp
-Wire Wire Line
-	5450 1600 7650 1600
-Connection ~ 5500 1600
-Wire Wire Line
-	5500 1200 5500 1600
-Wire Wire Line
-	5750 1100 5450 1100
-Wire Wire Line
-	7650 1100 6450 1100
-Connection ~ 7650 1600
 $Comp
 L GND #PWR?
@@
 	1    0    0    -1
 $EndComp
-Connection ~ 7650 2100
-Connection ~ 7650 1100
 $Comp
 L CRCW060310K0FKEA R?
@@
 	0    1    1    0
 $EndComp
-Connection ~ 2650 1800
-Connection ~ 2150 1900
 $Comp
 L +3.3V #PWR?
@@
 	1    0    0    -1
 $EndComp
-Wire Wire Line
-	2150 2700 2150 2600
-Wire Wire Line
-	2650 1050 2650 1000
 Text Label 3050 1900 0    60   ~ 0
 BOOT0
@@
 Text Notes 650  1400 0    60   ~ 0
 BOOT0 = 0 - Flash\nBOOT0 = 1 - Bootloader
-Wire Wire Line
-	4250 1800 2650 1800
-Wire Wire Line
-	4250 1900 2150 1900
 $Comp
 L ABLS2-8.000MHZ-D4Y-T U?
@@
 	0    1    1    0
 $EndComp
-Wire Wire Line
-	5450 4500 5950 4500
-Wire Wire Line
-	5650 5400 6950 5400
-Wire Wire Line
-	6950 4400 6950 4850
-Wire Wire Line
-	5450 4400 6950 4400
-Wire Wire Line
-	6950 4500 6550 4500
-Connection ~ 6950 4500
-Wire Wire Line
-	6950 5250 6950 5500
 $Comp
 L GND #PWR?
@@
 	1    0    0    -1
 $EndComp
+$Comp
+L Header,7x1,2.54mm U?
+U 1 1 5786AD4A
+P 1550 6650
+F 0 "U?" H 1950 6600 60  0000 C CNN
+F 1 "Header,7x1,2.54mm" H 2100 7550 60  0000 C CNN
+F 2 "" H 1550 6650 60  0000 C CNN
+F 3 "" H 1550 6650 60  0000 C CNN
+	1    1550 6650
+	-1   0    0    1
+$EndComp
+Wire Wire Line
+	5500 5800 5500 5900
+Wire Wire Line
+	5500 5900 5500 6000
+Wire Wire Line
+	5500 6000 5500 6100
+Wire Wire Line
+	5500 6100 5500 6200
+Wire Wire Line
+	5500 6200 5500 6350
+Wire Wire Line
+	5500 5800 5450 5800
+Wire Wire Line
+	5450 6200 5500 6200
+Connection ~ 5500 6200
+Wire Wire Line
+	5450 6100 5500 6100
+Connection ~ 5500 6100
+Wire Wire Line
+	5450 6000 5500 6000
+Connection ~ 5500 6000
+Wire Wire Line
+	5450 5900 5500 5900
+Connection ~ 5500 5900
+Wire Wire Line
+	2650 1650 2650 1800
+Wire Wire Line
+	2650 1800 2650 2000
+Wire Wire Line
+	2650 2700 2650 2600
+Wire Wire Line
+	2150 1650 2150 1900
+Wire Wire Line
+	2150 1900 2150 2000
+Wire Wire Line
+	2150 1050 2150 1000
+Wire Wire Line
+	5500 1500 5450 1500
+Connection ~ 5500 1400
+Connection ~ 5500 1300
+Connection ~ 5500 1500
+Wire Wire Line
+	5500 1400 5450 1400
+Wire Wire Line
+	5450 1300 5500 1300
+Wire Wire Line
+	5450 1200 5500 1200
+Wire Wire Line
+	5650 1600 5650 1650
+Wire Wire Line
+	6150 1600 6150 1650
+Connection ~ 5650 1600
+Wire Wire Line
+	6650 1600 6650 1650
+Connection ~ 6150 1600
+Wire Wire Line
+	7150 1600 7150 1650
+Connection ~ 6650 1600
+Wire Wire Line
+	7650 1050 7650 1100
+Wire Wire Line
+	7650 1100 7650 1600
+Wire Wire Line
+	7650 1600 7650 1650
+Connection ~ 7150 1600
+Wire Wire Line
+	7650 2050 7650 2100
+Wire Wire Line
+	7650 2100 7650 2150
+Wire Wire Line
+	5650 2100 6150 2100
+Wire Wire Line
+	6150 2100 6650 2100
+Wire Wire Line
+	6650 2100 7150 2100
+Wire Wire Line
+	7150 2100 7650 2100
+Wire Wire Line
+	5650 2100 5650 2050
+Wire Wire Line
+	6150 2050 6150 2100
+Connection ~ 6150 2100
+Wire Wire Line
+	6650 2050 6650 2100
+Connection ~ 6650 2100
+Wire Wire Line
+	7150 2050 7150 2100
+Connection ~ 7150 2100
+Wire Wire Line
+	5450 1600 5500 1600
+Wire Wire Line
+	5500 1600 5650 1600
+Wire Wire Line
+	5650 1600 6150 1600
+Wire Wire Line
+	6150 1600 6650 1600
+Wire Wire Line
+	6650 1600 7150 1600
+Wire Wire Line
+	7150 1600 7650 1600
+Connection ~ 5500 1600
+Wire Wire Line
+	5500 1200 5500 1300
+Wire Wire Line
+	5500 1300 5500 1400
+Wire Wire Line
+	5500 1400 5500 1500
+Wire Wire Line
+	5500 1500 5500 1600
+Wire Wire Line
+	5750 1100 5450 1100
+Wire Wire Line
+	7650 1100 6450 1100
+Connection ~ 7650 1600
+Connection ~ 7650 2100
+Connection ~ 7650 1100
+Connection ~ 2650 1800
+Connection ~ 2150 1900
+Wire Wire Line
+	2150 2700 2150 2600
+Wire Wire Line
+	2650 1050 2650 1000
+Wire Wire Line
+	4250 1800 2650 1800
+Wire Wire Line
+	4250 1900 2150 1900
+Wire Wire Line
+	5450 4500 5650 4500
+Wire Wire Line
+	5650 4500 5950 4500
+Wire Wire Line
+	5650 5400 6950 5400
+Wire Wire Line
+	6950 4400 6950 4500
+Wire Wire Line
+	6950 4500 6950 4850
+Wire Wire Line
+	5450 4400 6950 4400
+Wire Wire Line
+	6950 4500 6550 4500
+Connection ~ 6950 4500
+Wire Wire Line
+	6950 5250 6950 5400
+Wire Wire Line
+	6950 5400 6950 5500
 Connection ~ 6950 5400
 Wire Wire Line
@@
 Wire Wire Line
 	5650 5400 5650 5250
+Wire Wire Line
+	1550 7250 2600 7250
+Wire Wire Line
+	1550 7150 2600 7150
+Wire Wire Line
+	1550 7050 2600 7050
+Wire Wire Line
+	1550 6950 2600 6950
+Wire Wire Line
+	1550 6850 2600 6850
+Wire Wire Line
+	1550 6750 2600 6750
+Wire Wire Line
+	4250 3600 3200 3600
+Wire Wire Line
+	4250 3700 3200 3700
+Wire Wire Line
+	4250 3800 3200 3800
+Wire Wire Line
+	4250 4300 3200 4300
+Wire Wire Line
+	4250 4400 3200 4400
+Text Label 3250 3600 0    60   ~ 0
+SYS_JTMS-SWDIO
+Text Label 3250 3700 0    60   ~ 0
+SYS_JTCK-SWCLK
+Text Label 3250 3800 0    60   ~ 0
+SYS_JTDI
+Text Label 3250 4300 0    60   ~ 0
+SYS_JTDO-TRACESWO
+Text Label 3250 4400 0    60   ~ 0
+SYS_NJTRST
+$Comp
+L GND #PWR?
+U 1 1 5786C411
+P 1650 7450
+F 0 "#PWR?" H 1650 7200 50  0001 C CNN
+F 1 "GND" H 1650 7300 50  0000 C CNN
+F 2 "" H 1650 7450 50  0000 C CNN
+F 3 "" H 1650 7450 50  0000 C CNN
+	1    1650 7450
+	1    0    0    -1
+$EndComp
+Wire Wire Line
+	1650 7450 1650 7350
+Wire Wire Line
+	1650 7350 1550 7350
+Text Label 1600 7250 0    60   ~ 0
+SYS_JTMS-SWDIO
+Text Label 1600 7150 0    60   ~ 0
+SYS_JTCK-SWCLK
+Text Label 1600 7050 0    60   ~ 0
+SYS_JTDO-TRACESWO
+Text Label 1600 6950 0    60   ~ 0
+NRST
+Text Label 1600 6850 0    60   ~ 0
+SYS_JTDI
+Text Label 1600 6750 0    60   ~ 0
+SYS_NJTRST
 $EndSCHEMATC

Commit message: added debug header and updated pin mux
Parts:
- added U?: Header,3x1,2.54mm, symbol Header,3x1,2.54mm
Connections:
- net labels added: USART1_RX_DEBUG, USART1_TX_DEBUG
- wire segments 77 -> 83
Other:
- note added: "DEBUG USART\n(Place net names in silk)"
- note added: "Programming header\n(Place net names in silk)"
- note added: "RX/TX relative to processor"
Changed lines of the file:
@@
 Text Label 1600 6750 0    60   ~ 0
 SYS_NJTRST
+$Comp
+L Header,3x1,2.54mm U?
+U 1 1 5786B8E8
+P 4100 7000
+F 0 "U?" H 4500 7000 60  0000 C CNN
+F 1 "Header,3x1,2.54mm" H 4750 7550 60  0000 C CNN
+F 2 "" H 4100 7000 60  0000 C CNN
+F 3 "" H 4100 7000 60  0000 C CNN
+	1    4100 7000
+	-1   0    0    1
+$EndComp
+Wire Wire Line
+	4100 7150 5050 7150
+Wire Wire Line
+	4100 7250 5050 7250
+Wire Wire Line
+	5450 3000 6500 3000
+Text Label 5500 3000 0    60   ~ 0
+USART1_RX_DEBUG
+Wire Wire Line
+	5450 2900 6500 2900
+Text Label 5500 2900 0    60   ~ 0
+USART1_TX_DEBUG
+$Comp
+L GND #PWR?
+U 1 1 5786D4A1
+P 4200 7450
+F 0 "#PWR?" H 4200 7200 50  0001 C CNN
+F 1 "GND" H 4200 7300 50  0000 C CNN
+F 2 "" H 4200 7450 50  0000 C CNN
+F 3 "" H 4200 7450 50  0000 C CNN
+	1    4200 7450
+	1    0    0    -1
+$EndComp
+Wire Wire Line
+	4200 7450 4200 7350
+Wire Wire Line
+	4200 7350 4100 7350
+Text Label 4150 7250 0    60   ~ 0
+USART1_RX_DEBUG
+Text Label 4150 7150 0    60   ~ 0
+USART1_TX_DEBUG
+Text Notes 1350 6500 0    60   ~ 0
+Programming header\n(Place net names in silk)
+Text Notes 3900 6900 0    60   ~ 0
+DEBUG USART\n(Place net names in silk)
+Text Notes 6850 3000 0    60   ~ 0
+RX/TX relative to processor
 $EndSCHEMATC

Commit message: added arduino style headers
Parts:
- added CN? (x2): Header,8x1,2.54mm, symbol Header,8x1,2.54mm
- added CN?: Header,6x1,2.54mm, symbol Header,6x1,2.54mm
- added CN?: Header,10x1,2.54mm, symbol Header,10x1,2.54mm
Connections:
- wire segments 83 -> 60
Changed lines of the file:
@@
 LIBS:header-7x1-254
 LIBS:header-3x1-254
+LIBS:header-8x1-254
+LIBS:header-6x1-254
+LIBS:header-10x1-254
 LIBS:osps-cache
 EELAYER 25 0
@@
 $EndComp
 Wire Wire Line
-	5500 5800 5500 5900
-Wire Wire Line
-	5500 5900 5500 6000
-Wire Wire Line
-	5500 6000 5500 6100
-Wire Wire Line
-	5500 6100 5500 6200
-Wire Wire Line
-	5500 6200 5500 6350
+	5500 5800 5500 6350
 Wire Wire Line
 	5500 5800 5450 5800
@@
 Connection ~ 5500 5900
 Wire Wire Line
-	2650 1650 2650 1800
-Wire Wire Line
-	2650 1800 2650 2000
+	2650 1650 2650 2000
 Wire Wire Line
 	2650 2700 2650 2600
 Wire Wire Line
-	2150 1650 2150 1900
-Wire Wire Line
-	2150 1900 2150 2000
+	2150 1650 2150 2000
 Wire Wire Line
 	2150 1050 2150 1000
@@
 Connection ~ 6650 1600
 Wire Wire Line
-	7650 1050 7650 1100
-Wire Wire Line
-	7650 1100 7650 1600
-Wire Wire Line
-	7650 1600 7650 1650
+	7650 1050 7650 1650
 Connection ~ 7150 1600
 Wire Wire Line
-	7650 2050 7650 2100
-Wire Wire Line
-	7650 2100 7650 2150
-Wire Wire Line
-	5650 2100 6150 2100
-Wire Wire Line
-	6150 2100 6650 2100
-Wire Wire Line
-	6650 2100 7150 2100
-Wire Wire Line
-	7150 2100 7650 2100
+	7650 2050 7650 2150
+Wire Wire Line
+	5650 2100 7650 2100
 Wire Wire Line
 	5650 2100 5650 2050
@@
 Connection ~ 7150 2100
 Wire Wire Line
-	5450 1600 5500 1600
-Wire Wire Line
-	5500 1600 5650 1600
-Wire Wire Line
-	5650 1600 6150 1600
-Wire Wire Line
-	6150 1600 6650 1600
-Wire Wire Line
-	6650 1600 7150 1600
-Wire Wire Line
-	7150 1600 7650 1600
+	5450 1600 7650 1600
 Connection ~ 5500 1600
 Wire Wire Line
-	5500 1200 5500 1300
-Wire Wire Line
-	5500 1300 5500 1400
-Wire Wire Line
-	5500 1400 5500 1500
-Wire Wire Line
-	5500 1500 5500 1600
+	5500 1200 5500 1600
 Wire Wire Line
 	5750 1100 5450 1100
@@
 	4250 1900 2150 1900
 Wire Wire Line
-	5450 4500 5650 4500
-Wire Wire Line
-	5650 4500 5950 4500
+	5450 4500 5950 4500
 Wire Wire Line
 	5650 5400 6950 5400
 Wire Wire Line
-	6950 4400 6950 4500
-Wire Wire Line
-	6950 4500 6950 4850
+	6950 4400 6950 4850
 Wire Wire Line
 	5450 4400 6950 4400
@@
 Connection ~ 6950 4500
 Wire Wire Line
-	6950 5250 6950 5400
-Wire Wire Line
-	6950 5400 6950 5500
+	6950 5250 6950 5500
 Connection ~ 6950 5400
 Wire Wire Line
@@
 Text Notes 6850 3000 0    60   ~ 0
 RX/TX relative to processor
+$Comp
+L Header,8x1,2.54mm CN?
+U 1 1 5787EC1C
+P 9000 4100
+F 0 "CN?" H 9300 5000 60  0000 C CNN
+F 1 "Header,8x1,2.54mm" H 9000 3950 60  0000 C CNN
+F 2 "" H 9000 4100 60  0000 C CNN
+F 3 "" H 9000 4100 60  0000 C CNN
+	1    9000 4100
+	1    0    0    -1
+$EndComp
+$Comp
+L Header,8x1,2.54mm CN?
+U 1 1 5787EE1A
+P 10100 4450
+F 0 "CN?" H 10500 4350 60  0000 C CNN
+F 1 "Header,8x1,2.54mm" H 10100 5400 60  0000 C CNN
+F 2 "" H 10100 4450 60  0000 C CNN
+F 3 "" H 10100 4450 60  0000 C CNN
+	1    10100 4450
+	-1   0    0    1
+$EndComp
+$Comp
+L Header,6x1,2.54mm CN?
+U 1 1 5787F901
+P 9000 5650
+F 0 "CN?" H 9300 6750 60  0000 C CNN
+F 1 "Header,6x1,2.54mm" H 9050 5900 60  0000 C CNN
+F 2 "" H 9000 5650 60  0000 C CNN
+F 3 "" H 9000 5650 60  0000 C CNN
+	1    9000 5650
+	1    0    0    -1
+$EndComp
+$Comp
+L Header,10x1,2.54mm CN?
+U 1 1 5787FA71
+P 10100 2650
+F 0 "CN?" H 10450 3000 60  0000 C CNN
+F 1 "Header,10x1,2.54mm" H 10100 4200 60  0000 C CNN
+F 2 "" H 10100 2650 60  0000 C CNN
+F 3 "" H 10100 2650 60  0000 C CNN
+	1    10100 2650
+	-1   0    0    1
+$EndComp
 $EndSCHEMATC

Commit message: wire up headrer as on dev board
Connections:
- net labels added: +3.3VADC, PA0, PA1, PA10, PA2, PA3, PA4, PA8, PA9, PB0, PB13, PB14, PB15, PB5, PB6, PB8, PB9, PC0, PC1, PC7
- wire segments 60 -> 110
- no-connect marks 0 -> 1
Other:
- note added: "Arduino style headers"
