File: DesignDocuments/osps/processor.sch (KiCad schematic (older format))
At the start: 20 parts

Commit message: staredt UI sheet and moved USART
Connections:
- net labels added: PA2_USART2_TX, PA3_USART2_RX
- net labels removed: PA2, PA3
Changed lines of the file:
@@
 $Descr A4 11693 8268
 encoding utf-8
-Sheet 2 2
+Sheet 2 3
 Title ""
 Date ""
@@
 Wire Wire Line
 	4200 7350 4100 7350
-Text Label 4150 7250 0    60   ~ 0
-USART1_RX_DEBUG
-Text Label 4150 7150 0    60   ~ 0
-USART1_TX_DEBUG
 Text Notes 1350 6500 0    60   ~ 0
 Programming header\n(Place net names in silk)
@@
 Wire Wire Line
 	8800 3900 7750 3900
-Text Label 9950 5550 0    60   ~ 0
-PA3
-Text Label 9950 5450 0    60   ~ 0
-PA2
 Text Label 9950 5350 0    60   ~ 0
 PA10
@@
 Text Label 5500 2500 0    60   ~ 0
 PC0
-Text Label 3250 2600 0    60   ~ 0
-PA3
-Text Label 3250 2500 0    60   ~ 0
-PA2
 Text Label 3250 3300 0    60   ~ 0
 PA10
@@
 Text Label 3250 4800 0    60   ~ 0
 PB8
+Text Label 3250 2500 0    60   ~ 0
+PA2_USART2_TX
+Text Label 3250 2600 0    60   ~ 0
+PA3_USART2_RX
+Text Label 4150 7150 0    60   ~ 0
+PA2_USART2_TX
+Text Label 4150 7250 0    60   ~ 0
+PA3_USART2_RX
+Text Label 9950 5450 0    60   ~ 0
+PA2_USART2_TX
+Text Label 9950 5550 0    60   ~ 0
+PA3_USART2_RX
 $EndSCHEMATC

Commit message: added display to mcu pinout with connector
Connections:
- net labels added: PA13_SYS_JTMS-SWDIO, PA14_SYS_JTCK-SWCLK, PA15_SYS_JTDI, PA8_DISP_RS, PB14_DISP_DB4, PB15_DISP_DB5, PB3_SYS_JTDO-TRACESWO, PB4_SYS_NJTRST, PC6_DISP_DB6, PC7_DISP_DB7, PC8_DISP_E, PC9_DISP_RW
- net labels removed: SYS_JTCK-SWCLK, SYS_JTDI, SYS_JTMS-SWDIO, USART1_RX_DEBUG, USART1_TX_DEBUG
- wire segments 110 -> 113
Other:
- moved on the sheet: R?
